Commit message: Add Gazebo9 Support

File: motoman/motoman_mh5_support/urdf/mh5.xacro (robot description, xacro)
@@ -3,3 +3,7 @@
 	<xacro:include filename="$(find motoman_mh5_support)/urdf/mh5_macro.xacro" />
 	<xacro:motoman_mh5 prefix=""/>
+	<!-- .......... NEWLY ADDED BY ADAM .............. -->
+	<xacro:include filename="$(find motoman_mh5_support)/urdf/mh5.gazebo">
+		<arg name="prefix" value="${prefix}" />
+	</xacro:include>
 </robot>

File: motoman/motoman_mh5_support/urdf/mh5_macro.xacro (robot description, xacro)
@@ -3,4 +3,5 @@
 	<xacro:macro name="motoman_mh5" params="prefix">
 		<!-- link list -->
+		<link name="world"/>  		<!-- ADDED NEW: World Link-->
 		<link name="${prefix}base_link">
 			<visual>
@@ -22,4 +23,12 @@
 				</material>
 			</collision>
+			<inertial>
+	      <origin xyz="0 0 0.1" rpy="0 0 0"/>
+	      <mass value="1"/>
+	      <inertia
+	        ixx="0.0077" ixy="0.0" ixz="0.0"
+	        iyy="0.0066" iyz="0.0"
+	        izz="0.0077"/>
+	    </inertial>
 		</link>
 		<link name="${prefix}link_s">
@@ -38,4 +47,12 @@
 				<material name="yellow"/>
 			</collision>
+			<inertial>
+	      <origin xyz="0 0 0.05" rpy="0 0 0"/>
+	      <mass value="1"/>
+	      <inertia
+	        ixx="0.0052" ixy="0.0" ixz="0.0"
+	        iyy="0.0052" iyz="0.0"
+	        izz="0.0066"/>
+	    </inertial>
 		</link>
 		<link name="${prefix}link_l">
@@ -54,4 +71,12 @@
 				<material name="yellow"/>
 			</collision>
+			<inertial>
+	      <origin xyz="0 0 0.13" rpy="0 0 0"/>
+	      <mass value="1"/>
+	      <inertia
+	        ixx="0.02055" ixy="0.0" ixz="0.0"
+	        iyy="0.01875" iyz="0.0"
+	        izz="0.00555"/>
+	    </inertial>
 		</link>
 		<link name="${prefix}link_u">
@@ -70,4 +95,12 @@
 				<material name="yellow"/>
 			</collision>
+			<inertial>
+	      <origin xyz="0 0 0.05" rpy="0 0 0"/>
+	      <mass value="1"/>
+	      <inertia
+	        ixx="0.00328" ixy="0.0" ixz="0.0"
+	        iyy="0.00354" iyz="0.0"
+	        izz="0.00401"/>
+	    </inertial>
 		</link>
 		<link name="${prefix}link_r">
@@ -86,4 +119,12 @@
 				<material name="yellow"/>
 			</collision>
+			<inertial>
+	      <origin xyz="0.1 0 0" rpy="0 0 0"/>
+	      <mass value="1"/>
+	      <inertia
+	        ixx="0.00184" ixy="0.0" ixz="0.0"
+	        iyy="0.00708" iyz="0.0"
+	        izz="0.00691"/>
+	    </inertial>
 		</link>
 		<link name="${prefix}link_b">
@@ -102,4 +143,12 @@
 				<material name="yellow"/>
 			</collision>
+			<inertial>
+	      <origin xyz="0.05 0 0" rpy="0 0 0"/>
+	      <mass value="1"/>
+	      <inertia
+	        ixx="0.000708" ixy="0.0" ixz="0.0"
+	        iyy="0.001308" iyz="0.0"
+	        izz="0.004167"/>
+	    </inertial>
 		</link>
 		<link name="${prefix}link_t">
@@ -116,7 +165,19 @@
 				<material name="yellow"/>
 			</collision>
+			<inertial>
+	      <origin xyz="0 0 0" rpy="0 0 0"/>
+	      <mass value="1"/>
+	      <inertia
+	        ixx="0.00041667" ixy="0.0" ixz="0.0"
+	        iyy="0.00028333" iyz="0.0"
+	        izz="0.00028333"/>
+	    </inertial>
 		</link>
 		<!-- end of link list -->
 		<!-- joint list -->
+		<joint name="fixed" type="fixed">  <!-- ADDED BY ADAM:: Start -->
+			<parent link="world"/>
+			<child link="${prefix}base_link"/>
+		</joint>               		         <!-- ADDED BY ADAM:: END -->
 		<joint name="${prefix}joint_s" type="revolute">
 			<parent link="${prefix}base_link"/>
@@ -142,5 +203,6 @@
            won't hit link_l even when joint_r is at 45 degrees.  The
            old limits were converted directly from the MH5 data sheet,
-           which was clearly way off. -->
+           which was clearly way off.
+				  .. Noted by Adam Buynak February 2020 -->
 			<limit lower="-1.0122" upper="3.2218" effort="100" velocity="2.96" />
 		</joint>
