Commit message: Annotation Added

File: motoman/motoman_mh5_support/urdf/mh5_macro.xacro (robot description, xacro)
@@ -3,5 +3,5 @@
 	<xacro:macro name="motoman_mh5" params="prefix">
 		<!-- link list -->
-		<link name="world"/>  		<!-- ADDED NEW: World Link-->
+		<link name="world"/>  		<!-- ADDED NEW: World Link. Required for robot to be rigidly attached to world.-->
 		<link name="${prefix}base_link">
 			<visual>
