Commit message: Generate MoveIt Package for MH5 + PGN64 grippers
Build MoveIt package for MH5 with the PGN64 parallel grippers. 
Gripper added as an extension of final link_t. Did NOT implement as an 
end effector within MoveIt.
-- Singular Kinematic Chain. Fixed joints between link_t, eef_0, and 
eef_tcp.
-- No control of eef built into package.

File: schunk_pgn64_support/urdf/pgn64_macro.xacro (robot description, xacro)
@@ -42,5 +42,11 @@
 			<child link="${prefix}tcp"/>
 		</joint>
-		<link name="${prefix}tcp"/>
+		<link name="${prefix}tcp">
+			<visual>
+				<geometry>
+					<sphere radius="0.005"/>
+				</geometry>
+			</visual>
+		</link>
 	</xacro:macro>
 </robot>
