Commit message: Remove "robot_" prefix on Joints
* Changes driven by discussion on PR#7 w/ hansen95 *

**Notable Changes**
- Remove "robot_" prefix on robot joints.
  Retained "eef_" prefix on end effectors
- Update controllers.yaml to remove robot prefix
- Set join name yaml file to motoman_mh5_support/config/____.yaml

Kept planning group name as "mh5_arm" per original PR #7

File: schunk_pgn64_support/urdf/mh5_with_pgn64_macro.xacro (robot description, xacro)
@@ -7,17 +7,17 @@
   <xacro:macro name="motoman_mh5_with_pgn64" params="prefix">
     <!-- Instantiate MH5 robot and PGN64 eef model -->
-    <xacro:motoman_mh5 	prefix="${prefix}robot_" />
+    <xacro:motoman_mh5 	prefix="${prefix}" />
     <xacro:schunk_pgn64	prefix="${prefix}eef_" />
     <!-- Attach eef to MH5 model -->
     <!-- Note: this assumes that the 'schunk_pgn64' macro defines a 'tool0'
          link which is the start of it's kinematic chain (if any) -->
-    <joint name="${prefix}robot_flange-${prefix}eef_tool0" type="fixed">
+    <joint name="${prefix}flange-${prefix}eef_tool0" type="fixed">
       <origin xyz="0 0 0" rpy="0 0 0" />
-      <parent link="${prefix}robot_link_t" />
+      <parent link="${prefix}link_t" />
       <child link="${prefix}eef_tool0" />
     </joint>
     <!-- .......... GAZEBO SUPPORT .............. -->
   	<xacro:include filename="$(find motoman_mh5_support)/urdf/mh5.gazebo">
-  		<arg name="prefix" value="${prefix}robot_" />
+  		<arg name="prefix" value="${prefix}" />
   	</xacro:include>
   	<xacro:include filename="$(find schunk_pgn64_support)/urdf/pgn64.gazebo">
