Commit message: Corrected MS210 URDF
Estimated joint transforms through estimating the position in rviz. 
Guessing accuracy of 2-3 decimal precision. Highly suggest confirming 
values and improving precision with "SW to URDF" converter.

Updated STL's to place each STL's origin coincident with the rotational 
joint nearest to the base of the robot. This allows a simple transform 
from lower connection point to the next link's origin.

All changes intented to meet ROS Industrial Robot URDF guide.

File: motoman_ms210_support/urdf/ms210_macro.xacro (robot description, xacro)
@@ -142,5 +142,5 @@
     <parent link="${prefix}base_link" />
     <child  link="${prefix}link_s" />
-    <origin xyz="0 -0.262 0" rpy="1.5708 -0.021404 0" />
+    <origin xyz="0 0 0.342" rpy="0 0 0" />
     <axis   xyz="0 0 1" />
     <limit
@@ -153,6 +153,6 @@
     <parent link="${prefix}link_s" />
     <child link="${prefix}link_l" />
-    <origin xyz="0.015747 0 -0.26964" rpy="0 -0.024083 0" />
-    <axis xyz="0 0 0" />
+    <origin xyz="0.325 0 0.333" rpy="0 0 0" />
+    <axis xyz="0 1 0" />
     <limit
       lower="-1.0472"
@@ -164,5 +164,5 @@
     <parent link="${prefix}link_l" />
     <child link="${prefix}link_u" />
-    <origin xyz="0.325 -0.00021402 1.8" rpy="0 0.46111 0" />
+    <origin xyz="0 0 1.15" rpy="0 0 0" />
     <axis xyz="0 1 0" />
     <limit
@@ -175,5 +175,5 @@
     <parent link="${prefix}link_u" />
     <child link="${prefix}link_r" />
-    <origin xyz="1.0365 0.00021402 0.3" rpy="0.0094618 0 0" />
+    <origin xyz="0.9735 0 0.3" rpy="0 0 0" />
     <axis xyz="1 0 0" />
     <limit
@@ -184,5 +184,5 @@
   </joint>
   <joint name="${prefix}joint_b" type="revolute">
-    <origin xyz="0.18851 0 0" rpy="0 -0.18526 0" />
+    <origin xyz="0.2515 0 0" rpy="0 0 0" />
     <parent link="${prefix}link_r" />
     <child link="${prefix}link_b" />
@@ -195,5 +195,5 @@
   </joint>
   <joint name="${prefix}joint_t" type="revolute">
-    <origin xyz="0.21566 0 0" rpy="-1.5749 0 0" />
+    <origin xyz="0.21695 0 0" rpy="0 0 0" />
     <parent link="${prefix}link_b" />
     <child link="${prefix}link_t" />
